Commit message: Add odometry calibration bringup and update robot configuration

File: urdf/experiment_robot.urdf.xacro (robot description, xacro)
@@ -24,5 +24,6 @@
     <link name="${side}_wheel_link">
       <visual>
-        <origin xyz="0 0 ${wheel_radius}" rpy="1.57079632679 0 0"/>
+        <!-- The wheel link origin is its axle center. -->
+        <origin xyz="0 0 0" rpy="1.57079632679 0 0"/>
         <geometry><cylinder radius="${wheel_radius}" length="${wheel_width}"/></geometry>
         <material name="wheel_black"/>
@@ -31,5 +32,5 @@
     <joint name="${side}_wheel_joint" type="fixed">
       <parent link="base_link"/><child link="${side}_wheel_link"/>
-      <origin xyz="0 ${y} 0" rpy="0 0 0"/>
+      <origin xyz="0 ${y} ${wheel_radius}" rpy="0 0 0"/>
     </joint>
   </xacro:macro>

Commit message: Integrate LiDAR navigation and resilient odometry fusion

File: urdf/experiment_robot.urdf.xacro (robot description, xacro)
@@ -67,4 +67,11 @@
     <parent link="base_link"/><child link="safety_footprint_link"/>
   </joint>
+  <!-- RPLIDAR S1 scan origin (rotating laser axis), not its bottom mounting face.
+       Measured from base_link: 8 mm forward, centered, 192 mm above ground. -->
+  <link name="laser"/>
+  <joint name="laser_joint" type="fixed">
+    <parent link="base_link"/><child link="laser"/>
+    <origin xyz="0.008 0 0.192" rpy="0 0 0"/>
+  </joint>
   <!-- Camera mounting reference is now on the robot centerline (y=0).
        Previous longitudinal position and mounting height are retained. -->

Commit message: backup

File: urdf/experiment_robot.urdf.xacro (robot description, xacro)
@@ -72,5 +72,6 @@
   <joint name="laser_joint" type="fixed">
     <parent link="base_link"/><child link="laser"/>
-    <origin xyz="0.008 0 0.192" rpy="0 0 0"/>
+    <!-- The scanner's +X direction faces the rear of the vehicle. -->
+    <origin xyz="0.008 0 0.192" rpy="0 0 ${pi}"/>
   </joint>
   <!-- Camera mounting reference is now on the robot centerline (y=0).

Commit message: Rename package to experiment_cat and integrate emcl2 localization

File: urdf/experiment_robot.urdf.xacro (robot description, xacro)
@@ -90,5 +90,5 @@
       <origin xyz="0 0 0" rpy="0 0 0"/>
       <!-- Ellipsoid: diameter 0.160, height 0.050; reference at its center. -->
-      <geometry><mesh filename="package://experiment_nav2/meshes/antenna.stl"/></geometry>
+      <geometry><mesh filename="package://experiment_cat/meshes/antenna.stl"/></geometry>
       <material name="antenna_white"/>
     </visual>
